File: hardware/kicad/C64Ethernet_M1_2N_legacy_capture.sch (KiCad schematic (older format))
At the start: 7 parts, among them J1 C64_USERPORT, J2 RJ45_MAGJACK, U1 LC4032V-5TN48C, U2 W5500, U3 REG_3V3, X1 25MHz

Commit message: fix: anchor schematic net labels with wire stubs
Connections:
- wire segments 0 -> 45
Other:
- note added: "M1.2N capture: labels are anchored through explicit wire stubs for deterministic KiCad migration/ERC connectivity."
- note removed: "M1.2N capture: labels are anchored directly to symbol pins for deterministic KiCad migration/ERC connectivity."
Changed lines of the file:
@@
 W5500 ETHERNET
 Text Notes 900 6750 0 60 ~ 12
-M1.2N capture: labels are anchored directly to symbol pins for deterministic KiCad migration/ERC connectivity.
+M1.2N capture: labels are anchored through explicit wire stubs for deterministic KiCad migration/ERC connectivity.
 $Comp
 L C64_USERPORT J1
@@
 	1 0 0 -1
 $EndComp
-Text Label 2500 3000 0 50 ~ 0
+Wire Wire Line
+	2500 3000 2600 3000
+Text Label 2600 3000 0 50 ~ 0
 PB0
-Text Label 2500 3100 0 50 ~ 0
+Wire Wire Line
+	2500 3100 2600 3100
+Text Label 2600 3100 0 50 ~ 0
 PB1
-Text Label 2500 3200 0 50 ~ 0
+Wire Wire Line
+	2500 3200 2600 3200
+Text Label 2600 3200 0 50 ~ 0
 PB2
-Text Label 2500 3300 0 50 ~ 0
+Wire Wire Line
+	2500 3300 2600 3300
+Text Label 2600 3300 0 50 ~ 0
 PB3
-Text Label 2500 3400 0 50 ~ 0
+Wire Wire Line
+	2500 3400 2600 3400
+Text Label 2600 3400 0 50 ~ 0
 PB4
-Text Label 2500 3500 0 50 ~ 0
+Wire Wire Line
+	2500 3500 2600 3500
+Text Label 2600 3500 0 50 ~ 0
 PB5
-Text Label 2500 3600 0 50 ~ 0
+Wire Wire Line
+	2500 3600 2600 3600
+Text Label 2600 3600 0 50 ~ 0
 PB6
-Text Label 2500 3700 0 50 ~ 0
+Wire Wire Line
+	2500 3700 2600 3700
+Text Label 2600 3700 0 50 ~ 0
 PB7
-Text Label 2500 3900 0 50 ~ 0
+Wire Wire Line
+	2500 3900 2600 3900
+Text Label 2600 3900 0 50 ~ 0
 PA2_HOST_STROBE
-Text Label 2500 4000 0 50 ~ 0
+Wire Wire Line
+	2500 4000 2600 4000
+Text Label 2600 4000 0 50 ~ 0
 DEVICE_IRQ
-Text Label 3900 2900 2 50 ~ 0
+Wire Wire Line
+	3900 2900 3800 2900
+Text Label 3800 2900 2 50 ~ 0
 PB0
-Text Label 3900 3000 2 50 ~ 0
+Wire Wire Line
+	3900 3000 3800 3000
+Text Label 3800 3000 2 50 ~ 0
 PB1
-Text Label 3900 3100 2 50 ~ 0
+Wire Wire Line
+	3900 3100 3800 3100
+Text Label 3800 3100 2 50 ~ 0
 PB2
-Text Label 3900 3200 2 50 ~ 0
+Wire Wire Line
+	3900 3200 3800 3200
+Text Label 3800 3200 2 50 ~ 0
 PB3
-Text Label 3900 3300 2 50 ~ 0
+Wire Wire Line
+	3900 3300 3800 3300
+Text Label 3800 3300 2 50 ~ 0
 PB4
-Text Label 3900 3400 2 50 ~ 0
+Wire Wire Line
+	3900 3400 3800 3400
+Text Label 3800 3400 2 50 ~ 0
 PB5
-Text Label 3900 3500 2 50 ~ 0
+Wire Wire Line
+	3900 3500 3800 3500
+Text Label 3800 3500 2 50 ~ 0
 PB6
-Text Label 3900 3600 2 50 ~ 0
+Wire Wire Line
+	3900 3600 3800 3600
+Text Label 3800 3600 2 50 ~ 0
 PB7
-Text Label 3900 3800 2 50 ~ 0
+Wire Wire Line
+	3900 3800 3800 3800
+Text Label 3800 3800 2 50 ~ 0
 PA2_HOST_STROBE
-Text Label 3900 3900 2 50 ~ 0
+Wire Wire Line
+	3900 3900 3800 3900
+Text Label 3800 3900 2 50 ~ 0
 DEVICE_IRQ
-Text Label 5500 2900 0 50 ~ 0
+Wire Wire Line
+	5500 2900 5600 2900
+Text Label 5600 2900 0 50 ~ 0
 SCLK
-Text Label 5500 3000 0 50 ~ 0
+Wire Wire Line
+	5500 3000 5600 3000
+Text Label 5600 3000 0 50 ~ 0
 MOSI
-Text Label 5500 3100 0 50 ~ 0
+Wire Wire Line
+	5500 3100 5600 3100
+Text Label 5600 3100 0 50 ~ 0
 MISO
-Text Label 5500 3200 0 50 ~ 0
+Wire Wire Line
+	5500 3200 5600 3200
+Text Label 5600 3200 0 50 ~ 0
 SCSn
-Text Label 5500 3300 0 50 ~ 0
+Wire Wire Line
+	5500 3300 5600 3300
+Text Label 5600 3300 0 50 ~ 0
 INTn
-Text Label 5500 3400 0 50 ~ 0
+Wire Wire Line
+	5500 3400 5600 3400
+Text Label 5600 3400 0 50 ~ 0
 RSTn
-Text Label 6900 2900 2 50 ~ 0
+Wire Wire Line
+	6900 2900 6800 2900
+Text Label 6800 2900 2 50 ~ 0
 SCLK
-Text Label 6900 3000 2 50 ~ 0
+Wire Wire Line
+	6900 3000 6800 3000
+Text Label 6800 3000 2 50 ~ 0
 MOSI
-Text Label 6900 3100 2 50 ~ 0
+Wire Wire Line
+	6900 3100 6800 3100
+Text Label 6800 3100 2 50 ~ 0
 MISO
-Text Label 6900 3200 2 50 ~ 0
+Wire Wire Line
+	6900 3200 6800 3200
+Text Label 6800 3200 2 50 ~ 0
 SCSn
-Text Label 6900 3300 2 50 ~ 0
+Wire Wire Line
+	6900 3300 6800 3300
+Text Label 6800 3300 2 50 ~ 0
 INTn
-Text Label 6900 3400 2 50 ~ 0
+Wire Wire Line
+	6900 3400 6800 3400
+Text Label 6800 3400 2 50 ~ 0
 RSTn
-Text Label 8500 2900 0 50 ~ 0
+Wire Wire Line
+	8500 2900 8600 2900
+Text Label 8600 2900 0 50 ~ 0
 EXRES1
-Text Label 8500 3100 0 50 ~ 0
+Wire Wire Line
+	8500 3100 8600 3100
+Text Label 8600 3100 0 50 ~ 0
 TXP
-Text Label 8500 3200 0 50 ~ 0
+Wire Wire Line
+	8500 3200 8600 3200
+Text Label 8600 3200 0 50 ~ 0
 TXN
-Text Label 8500 3400 0 50 ~ 0
+Wire Wire Line
+	8500 3400 8600 3400
+Text Label 8600 3400 0 50 ~ 0
 RXP
-Text Label 8500 3500 0 50 ~ 0
+Wire Wire Line
+	8500 3500 8600 3500
+Text Label 8600 3500 0 50 ~ 0
 RXN
-Text Label 9450 3200 2 50 ~ 0
+Wire Wire Line
+	9450 3200 9350 3200
+Text Label 9350 3200 2 50 ~ 0
 TXP
-Text Label 9450 3300 2 50 ~ 0
+Wire Wire Line
+	9450 3300 9350 3300
+Text Label 9350 3300 2 50 ~ 0
 TXN
-Text Label 9450 3500 2 50 ~ 0
+Wire Wire Line
+	9450 3500 9350 3500
+Text Label 9350 3500 2 50 ~ 0
 RXP
-Text Label 9450 3600 2 50 ~ 0
+Wire Wire Line
+	9450 3600 9350 3600
+Text Label 9350 3600 2 50 ~ 0
 RXN
-Text Label 6650 5400 2 50 ~ 0
+Wire Wire Line
+	6650 5400 6550 5400
+Text Label 6550 5400 2 50 ~ 0
 EXRES1
-Text Label 6950 5400 0 50 ~ 0
+Wire Wire Line
+	6950 5400 7050 5400
+Text Label 7050 5400 0 50 ~ 0
 GND
-Text Label 7450 5400 2 50 ~ 0
+Wire Wire Line
+	7450 5400 7350 5400
+Text Label 7350 5400 2 50 ~ 0
 OSC_RETURN
-Text Label 7750 5400 0 50 ~ 0
+Wire Wire Line
+	7750 5400 7850 5400
+Text Label 7850 5400 0 50 ~ 0
 OSC_RETURN
 $EndSCHEMATC

Commit message: revert: remove ERC wire stubs
Connections:
- wire segments 45 -> 0
Other:
- note added: "M1.2N capture: labels are anchored directly to symbol pins for deterministic KiCad migration/ERC connectivity."
- note removed: "M1.2N capture: labels are anchored through explicit wire stubs for deterministic KiCad migration/ERC connectivity."
Changed lines of the file:
@@
 W5500 ETHERNET
 Text Notes 900 6750 0 60 ~ 12
-M1.2N capture: labels are anchored through explicit wire stubs for deterministic KiCad migration/ERC connectivity.
+M1.2N capture: labels are anchored directly to symbol pins for deterministic KiCad migration/ERC connectivity.
 $Comp
 L C64_USERPORT J1
@@
 	1 0 0 -1
 $EndComp
-Wire Wire Line
-	2500 3000 2600 3000
-Text Label 2600 3000 0 50 ~ 0
+Text Label 2500 3000 0 50 ~ 0
 PB0
-Wire Wire Line
-	2500 3100 2600 3100
-Text Label 2600 3100 0 50 ~ 0
+Text Label 2500 3100 0 50 ~ 0
 PB1
-Wire Wire Line
-	2500 3200 2600 3200
-Text Label 2600 3200 0 50 ~ 0
+Text Label 2500 3200 0 50 ~ 0
 PB2
-Wire Wire Line
-	2500 3300 2600 3300
-Text Label 2600 3300 0 50 ~ 0
+Text Label 2500 3300 0 50 ~ 0
 PB3
-Wire Wire Line
-	2500 3400 2600 3400
-Text Label 2600 3400 0 50 ~ 0
+Text Label 2500 3400 0 50 ~ 0
 PB4
-Wire Wire Line
-	2500 3500 2600 3500
-Text Label 2600 3500 0 50 ~ 0
+Text Label 2500 3500 0 50 ~ 0
 PB5
-Wire Wire Line
-	2500 3600 2600 3600
-Text Label 2600 3600 0 50 ~ 0
+Text Label 2500 3600 0 50 ~ 0
 PB6
-Wire Wire Line
-	2500 3700 2600 3700
-Text Label 2600 3700 0 50 ~ 0
+Text Label 2500 3700 0 50 ~ 0
 PB7
-Wire Wire Line
-	2500 3900 2600 3900
-Text Label 2600 3900 0 50 ~ 0
+Text Label 2500 3900 0 50 ~ 0
 PA2_HOST_STROBE
-Wire Wire Line
-	2500 4000 2600 4000
-Text Label 2600 4000 0 50 ~ 0
+Text Label 2500 4000 0 50 ~ 0
 DEVICE_IRQ
-Wire Wire Line
-	3900 2900 3800 2900
-Text Label 3800 2900 2 50 ~ 0
+Text Label 3900 2900 2 50 ~ 0
 PB0
-Wire Wire Line
-	3900 3000 3800 3000
-Text Label 3800 3000 2 50 ~ 0
+Text Label 3900 3000 2 50 ~ 0
 PB1
-Wire Wire Line
-	3900 3100 3800 3100
-Text Label 3800 3100 2 50 ~ 0
+Text Label 3900 3100 2 50 ~ 0
 PB2
-Wire Wire Line
-	3900 3200 3800 3200
-Text Label 3800 3200 2 50 ~ 0
+Text Label 3900 3200 2 50 ~ 0
 PB3
-Wire Wire Line
-	3900 3300 3800 3300
-Text Label 3800 3300 2 50 ~ 0
+Text Label 3900 3300 2 50 ~ 0
 PB4
-Wire Wire Line
-	3900 3400 3800 3400
-Text Label 3800 3400 2 50 ~ 0
+Text Label 3900 3400 2 50 ~ 0
 PB5
-Wire Wire Line
-	3900 3500 3800 3500
-Text Label 3800 3500 2 50 ~ 0
+Text Label 3900 3500 2 50 ~ 0
 PB6
-Wire Wire Line
-	3900 3600 3800 3600
-Text Label 3800 3600 2 50 ~ 0
+Text Label 3900 3600 2 50 ~ 0
 PB7
-Wire Wire Line
-	3900 3800 3800 3800
-Text Label 3800 3800 2 50 ~ 0
+Text Label 3900 3800 2 50 ~ 0
 PA2_HOST_STROBE
-Wire Wire Line
-	3900 3900 3800 3900
-Text Label 3800 3900 2 50 ~ 0
+Text Label 3900 3900 2 50 ~ 0
 DEVICE_IRQ
-Wire Wire Line
-	5500 2900 5600 2900
-Text Label 5600 2900 0 50 ~ 0
+Text Label 5500 2900 0 50 ~ 0
 SCLK
-Wire Wire Line
-	5500 3000 5600 3000
-Text Label 5600 3000 0 50 ~ 0
+Text Label 5500 3000 0 50 ~ 0
 MOSI
-Wire Wire Line
-	5500 3100 5600 3100
-Text Label 5600 3100 0 50 ~ 0
+Text Label 5500 3100 0 50 ~ 0
 MISO
-Wire Wire Line
-	5500 3200 5600 3200
-Text Label 5600 3200 0 50 ~ 0
+Text Label 5500 3200 0 50 ~ 0
 SCSn
-Wire Wire Line
-	5500 3300 5600 3300
-Text Label 5600 3300 0 50 ~ 0
+Text Label 5500 3300 0 50 ~ 0
 INTn
-Wire Wire Line
-	5500 3400 5600 3400
-Text Label 5600 3400 0 50 ~ 0
+Text Label 5500 3400 0 50 ~ 0
 RSTn
-Wire Wire Line
-	6900 2900 6800 2900
-Text Label 6800 2900 2 50 ~ 0
+Text Label 6900 2900 2 50 ~ 0
 SCLK
-Wire Wire Line
-	6900 3000 6800 3000
-Text Label 6800 3000 2 50 ~ 0
+Text Label 6900 3000 2 50 ~ 0
 MOSI
-Wire Wire Line
-	6900 3100 6800 3100
-Text Label 6800 3100 2 50 ~ 0
+Text Label 6900 3100 2 50 ~ 0
 MISO
-Wire Wire Line
-	6900 3200 6800 3200
-Text Label 6800 3200 2 50 ~ 0
+Text Label 6900 3200 2 50 ~ 0
 SCSn
-Wire Wire Line
-	6900 3300 6800 3300
-Text Label 6800 3300 2 50 ~ 0
+Text Label 6900 3300 2 50 ~ 0
 INTn
-Wire Wire Line
-	6900 3400 6800 3400
-Text Label 6800 3400 2 50 ~ 0
+Text Label 6900 3400 2 50 ~ 0
 RSTn
-Wire Wire Line
-	8500 2900 8600 2900
-Text Label 8600 2900 0 50 ~ 0
+Text Label 8500 2900 0 50 ~ 0
 EXRES1
-Wire Wire Line
-	8500 3100 8600 3100
-Text Label 8600 3100 0 50 ~ 0
+Text Label 8500 3100 0 50 ~ 0
 TXP
-Wire Wire Line
-	8500 3200 8600 3200
-Text Label 8600 3200 0 50 ~ 0
+Text Label 8500 3200 0 50 ~ 0
 TXN
-Wire Wire Line
-	8500 3400 8600 3400
-Text Label 8600 3400 0 50 ~ 0
+Text Label 8500 3400 0 50 ~ 0
 RXP
-Wire Wire Line
-	8500 3500 8600 3500
-Text Label 8600 3500 0 50 ~ 0
+Text Label 8500 3500 0 50 ~ 0
 RXN
-Wire Wire Line
-	9450 3200 9350 3200
-Text Label 9350 3200 2 50 ~ 0
+Text Label 9450 3200 2 50 ~ 0
 TXP
-Wire Wire Line
-	9450 3300 9350 3300
-Text Label 9350 3300 2 50 ~ 0
+Text Label 9450 3300 2 50 ~ 0
 TXN
-Wire Wire Line
-	9450 3500 9350 3500
-Text Label 9350 3500 2 50 ~ 0
+Text Label 9450 3500 2 50 ~ 0
 RXP
-Wire Wire Line
-	9450 3600 9350 3600
-Text Label 9350 3600 2 50 ~ 0
+Text Label 9450 3600 2 50 ~ 0
 RXN
-Wire Wire Line
-	6650 5400 6550 5400
-Text Label 6550 5400 2 50 ~ 0
+Text Label 6650 5400 2 50 ~ 0
 EXRES1
-Wire Wire Line
-	6950 5400 7050 5400
-Text Label 7050 5400 0 50 ~ 0
+Text Label 6950 5400 0 50 ~ 0
 GND
-Wire Wire Line
-	7450 5400 7350 5400
-Text Label 7350 5400 2 50 ~ 0
+Text Label 7450 5400 2 50 ~ 0
 OSC_RETURN
-Wire Wire Line
-	7750 5400 7850 5400
-Text Label 7850 5400 0 50 ~ 0
+Text Label 7750 5400 0 50 ~ 0
 OSC_RETURN
 $EndSCHEMATC
