File: hardware/kicad/C64Ethernet.kicad_sch (KiCad schematic)
At the start: 0 parts

Commit message: M1.2j: establish native KiCad schematic connectivity baseline
Other:
- note added: "C64Ethernet native schematic connectivity baseline"
- note added: "CPLD: LC4032V-5TN48C reference; W5500: SPI + RSTn + INTn"
- note added: "ETHERNET: W5500 MDI -> magnetics/MagJack -> RJ45; ESD protection required"
- note added: "NOTE: This file is a connectivity baseline, not ERC-qualified production hardware."
- note added: "POWER: C64 +5V input -> protected 3.3V rail; W5500 EXRES1 12.4k 1%; 25MHz clock"
- note added: "USER PORT: PB0-PB7 bidirectional; PA2 HOST_STROBE; FLAG2 DEVICE_IRQ/READY"
Changed lines of the file:
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@@
-(kicad_sch (version 20231120) (generator eeschema)
+(kicad_sch (version 20231120) (generator c64ethernet-m0)
   (paper "A4")
+  (text "C64Ethernet native schematic connectivity baseline" (exclude_from_sim no) (at 100 40 0) (effects (font (size 1.27 1.27))))
+  (text "USER PORT: PB0-PB7 bidirectional; PA2 HOST_STROBE; FLAG2 DEVICE_IRQ/READY" (exclude_from_sim no) (at 100 50 0) (effects (font (size 1 1))))
+  (text "CPLD: LC4032V-5TN48C reference; W5500: SPI + RSTn + INTn" (exclude_from_sim no) (at 100 58 0) (effects (font (size 1 1))))
+  (text "POWER: C64 +5V input -> protected 3.3V rail; W5500 EXRES1 12.4k 1%; 25MHz clock" (exclude_from_sim no) (at 100 66 0) (effects (font (size 1 1))))
+  (text "ETHERNET: W5500 MDI -> magnetics/MagJack -> RJ45; ESD protection required" (exclude_from_sim no) (at 100 74 0) (effects (font (size 1 1))))
+  (text "NOTE: This file is a connectivity baseline, not ERC-qualified production hardware." (exclude_from_sim no) (at 100 82 0) (effects (font (size 1 1))))
   (sheet_instances (path "/" (page "1")))
 )

Commit message: hardware: promote migrated native KiCad schematic
Parts:
- added J1: C64_USERPORT, symbol C64_USERPORT
- added J2: RJ45_MAGJACK, symbol RJ45_MAGJACK
- added R1: 12.4k 1%, symbol R
- added U1: LC4032V-5TN48C, symbol LC4032V-5TN48C
- added U2: W5500, symbol W5500
- added U3: REG_3V3, symbol REG_3V3
- added X1: 25MHz, symbol CRYSTAL
Other:
- note added: "C64 USER PORT"
- note added: "LC4032V-5TN48C CPLD"
- note added: "M1.2N capture: labels are anchored directly to symbol pins for deterministic KiCad migration/ERC connectivity."
- note added: "W5500 ETHERNET"
- note removed: "C64Ethernet native schematic connectivity baseline"
- note removed: "CPLD: LC4032V-5TN48C reference; W5500: SPI + RSTn + INTn"
- note removed: "ETHERNET: W5500 MDI -> magnetics/MagJack -> RJ45; ESD protection required"
- note removed: "NOTE: This file is a connectivity baseline, not ERC-qualified production hardware."
- note removed: "POWER: C64 +5V input -> protected 3.3V rail; W5500 EXRES1 12.4k 1%; 25MHz clock"
- note removed: "USER PORT: PB0-PB7 bidirectional; PA2 HOST_STROBE; FLAG2 DEVICE_IRQ/READY"
- company: (none) -> Ploos-AS
- title: (none) -> C64Ethernet M1.2N engineering capture
