File: hardware/kicad/C64Ethernet.kicad_sch (KiCad schematic)
At the start: 7 parts, among them J1 C64_USERPORT, J2 RJ45_MAGJACK, U1 LC4032V-5TN48C, U2 W5500, U3 REG_3V3, X1 25MHz

Commit message: revert: restore native schematic ERC baseline
Other:
- note added: "M1.2N capture: labels are anchored directly to symbol pins for deterministic KiCad migration/ERC connectivity."
- note removed: "Native capture: explicit wires anchor previously dangling labels."
